File: PCB_Designs/ArduinoShieldDesign/ArduinoShieldDesign.kicad_sch (KiCad schematic)
At the start: 4 parts, among them J1 Power, J2 Digital/PWM, J3 Analog, J4 Digital/PWM

Commit message: PCB design
Parts:
- removed J1: Power, Connector_PinSocket_2.54mm:PinSocket_1x08_P2.54mm_Vertical, symbol Connector_Generic:Conn_01x08
- removed J2: Digital/PWM, Connector_PinSocket_2.54mm:PinSocket_1x10_P2.54mm_Vertical, symbol Connector_Generic:Conn_01x10
- removed J3: Analog, Connector_PinSocket_2.54mm:PinSocket_1x06_P2.54mm_Vertical, symbol Connector_Generic:Conn_01x06
- removed J4: Digital/PWM, Connector_PinSocket_2.54mm:PinSocket_1x08_P2.54mm_Vertical, symbol Connector_Generic:Conn_01x08
- added A1: Arduino_UNO_R3, Module:Arduino_UNO_R3, symbol MCU_Module:Arduino_UNO_R3
- added C1, C2, C3, C4, C5, C6, C7: 0.1 uF, Capacitor_SMD:CP_Elec_3x5.3, symbol Device:C
- added J1, J6: Conn_02x04_Odd_Even, Connector_IDC:IDC-Header_2x04_P2.54mm_Vertical, symbol Connector_Generic:Conn_02x04_Odd_Even
- added J2, J5: Screw_Terminal_01x05, TerminalBlock:TerminalBlock_Xinya_XY308-2.54-5P_1x05_P2.54mm_Horizontal, symbol Connector:Screw_Terminal_01x05
- added R1, R2, R3, R4: 1k, Resistor_SMD:R_0805_2012Metric_Pad1.20x1.40mm_HandSolder, symbol Device:R_US
- added U1: MCP3204, symbol Analog_ADC:MCP3204
- added U2, U3: MCP4922-EP, symbol Analog_DAC:MCP4922-EP
Connections:
- net +5V: now also A1.5 (+5V), C1.1, C2.1, C7.1, U1.13 (Vref), U1.14 (Vdd), U2.1 (VDD), U2.11 (VrefB), U3.1 (VDD), U3.11 (VrefB), U3.13 (VrefA)
- net GND: now also A1.29 (GND), A1.6 (GND), A1.7 (GND), C1.2, C2.2, C3.2, C4.2, C5.2, C6.2, C7.2, J1.2 (Pin_2), J1.4 (Pin_4), J1.6 (Pin_6), J1.8 (Pin_8), J2.5 (Pin_5), J5.5 (Pin_5), J6.2 (Pin_2), J6.4 (Pin_4), J6.6 (Pin_6), J6.8 (Pin_8), U1.12 (AGND), U1.7 (DGND), U2.12 (AVSS), U3.12 (AVSS)
- new net: J1.1 (Pin_1), J2.1 (Pin_1), R1.1
- new net: J1.3 (Pin_3), J2.2 (Pin_2), R2.1
- new net: J1.5 (Pin_5), J2.3 (Pin_3), R3.1
- new net: J1.7 (Pin_7), J2.4 (Pin_4), R4.1
- new net: J5.4 (Pin_4), J6.7 (Pin_7), U2.10 (VoutB)
- new net: J5.3 (Pin_3), J6.5 (Pin_5), U2.14 (VoutA)
- new net: C3.1, R1.2, U1.1 (CH0)
- new net: J5.1 (Pin_1), J6.1 (Pin_1), U3.14 (VoutA)
- new net: J5.2 (Pin_2), J6.3 (Pin_3), U3.10 (VoutB)
- new net: C5.1, R3.2, U1.3 (CH2)
- new net: C4.1, R2.2, U1.2 (CH1)
- new net: C6.1, R4.2, U1.4 (CH3)
- new net CIPO: A1.27 (D12), U1.10 (Dout)
- new net COPI: A1.26 (D11), U1.9 (Din), U2.5 (SDI), U3.5 (SDI)
- new net CS0: A1.25 (D10), U1.8 (~{CS}/SHDN)
- new net CS1: A1.24 (D9), U3.3 (~{CS})
- new net CS2: A1.23 (D8), U2.3 (~{CS})
- new net SCK: A1.28 (D13), U1.11 (CLK), U2.4 (SCK), U3.4 (SCK)
- new net nLDAC: A1.22 (D7), U2.8 (~{LDAC}), U3.8 (~{LDAC})
- new net nSHDN: A1.21 (D6), U2.9 (~{SHDN}), U3.9 (~{SHDN})
- no-connect marks 1 -> 0
